File: 01_KiCad_Project/dcs.kicad_pcb (KiCad board)
At the start: 4 copper layers, 62 x 45.9 mm, 50 parts, among them J1 PH2.0, J2 USB_C_Receptacle_USB2.0_16P, M1 12864 Display, Q1 2N7002, SW1 Push, SW3 TM-1011A, U1 E73-2G4M08S1C, U2 MCP73833, U3 TLV75533, U4 GSC1031YB-3V4000, U7 DRV2605L, U8 Ra-01SH

Commit message: Updated Gerbers and PCB
Routing:
- net GND: track 40.7 -> 40.0 mm
Changed lines of the file:
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@@
+	)
+	(segment
+		(start 210.95 127.25)
+		(end 210.95 127.95)
+		(width 0.2)
+		(layer "F.Cu")
+		(net "GND")
 	)
 	(segment
@@
 		(start 205.25 115.5125)
 		(end 205.25 116.6)
-		(width 0.4)
-		(layer "F.Cu")
-		(net "GND")
-	)
-	(segment
-		(start 217.05 118.5)
-		(end 216.4 117.85)
 		(width 0.4)
 		(layer "F.Cu")
@@
 	)
 	(segment
-		(start 217.05 118.9)
-		(end 217.05 118.5)
-		(width 0.4)
-		(layer "F.Cu")
-		(net "GND")
-	)
-	(segment
 		(start 194.2 94.65)
 		(end 195.55 94.65)
@@
 	)
 	(via
-		(at 217.05 118.9)
-		(size 0.6)
-		(drill 0.3)
-		(layers "F.Cu" "B.Cu")
-		(net "GND")
-	)
-	(via
 		(at 190.15 133.562055)
 		(size 0.6)
@@
 		(size 0.6)
 		(drill 0.3)
+		(layers "F.Cu" "B.Cu")
+		(net "GND")
+	)
+	(via
+		(at 210.95 127.95)
+		(size 0.6)
+		(drill 0.3)
